File: hardware/eCogs/eCog109_ISP_Programmer.sch (EAGLE design)
At the start: 2 parts

Commit message: Update eCogs to through hole
Parts:
- ECOG: value ECOG_BUSES_ROWECOG_BUSES_SMD -> ECOG_BUSES_ROWTHROUGHHOLE; device eCogs:ECOG_BUSES_ROWECOG_BUSES_SMD -> eCogs:ECOG_BUSES_ROWTHROUGHHOLE
Connections:
- net N$3: now also ECOG.RSV@B6; no longer ECOG.RESET@B6
Changed lines of the file:
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@@
 <parts>
 <part name="FRAME1" library="frames" deviceset="A3L-LOC" device=""/>
-<part name="ECOG" library="eCogs" deviceset="ECOG_BUSES_ROW" device="ECOG_BUSES_SMD" value="ECOG_BUSES_ROWECOG_BUSES_SMD"/>
+<part name="ECOG" library="eCogs" deviceset="ECOG_BUSES_ROW" device="THROUGHHOLE" value="ECOG_BUSES_ROWTHROUGHHOLE"/>
 <part name="GND1" library="eCogs" deviceset="GND" device=""/>
 <part name="3V3_PWR1" library="eCogs" deviceset="3V3" device=""/>
@@
 <net name="N$3" class="0">
 <segment>
-<pinref part="ECOG" gate="ECOG_BUSES" pin="RESET@B6"/>
+<pinref part="ECOG" gate="ECOG_BUSES" pin="RSV@B6"/>
 <wire x1="132.08" y1="149.86" x2="160.02" y2="149.86" width="0.2032" layer="91"/>
 <wire x1="160.02" y1="149.86" x2="160.02" y2="144.78" width="0.2032" layer="91"/>
