File: hardware/eCogs/eCog110_Buzzer.sch (EAGLE design)
At the start: 2 parts

Commit message: Update eCogs to through hole
Parts:
- ECOG: value ECOG_GENERAL_ROWECOG_GENERAL_SMD -> ECOG_GENERAL_ROWTHROUGHOLE; device eCogs:ECOG_GENERAL_ROWECOG_GENERAL_SMD -> eCogs:ECOG_GENERAL_ROWTHROUGHOLE
Changed lines of the file:
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@@
 <parts>
 <part name="FRAME1" library="frames" deviceset="A3L-LOC" device=""/>
-<part name="ECOG" library="eCogs" deviceset="ECOG_GENERAL_ROW" device="ECOG_GENERAL_SMD" value="ECOG_GENERAL_ROWECOG_GENERAL_SMD">
+<part name="ECOG" library="eCogs" deviceset="ECOG_GENERAL_ROW" device="THROUGHOLE" value="ECOG_GENERAL_ROWTHROUGHOLE">
 <attribute name="PARTNO" value="NREC010SABC-M30RC,SULLINS CONNECTOR SOLUTIONS,dk,S1013EC-10-ND,&quot;10 Positions Header, Unshrouded Connector 0.100&quot;&quot; (2.54mm) Surface Mount Tin eCog&quot;, REF78"/>
 </part>
