File: hardware/eCogs/eCog111_16ch_PWM_Servo.sch (EAGLE design)
At the start: 3 parts

Commit message: Update eCogs to through hole
Parts:
- ECOG: value ECOG_BUSES_ROWECOG_BUSES_SMD -> ECOG_BUSES_ROWTHROUGHHOLE; device eCogs:ECOG_BUSES_ROWECOG_BUSES_SMD -> eCogs:ECOG_BUSES_ROWTHROUGHHOLE
Changed lines of the file:
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@@
 <parts>
 <part name="FRAME1" library="frames" deviceset="A3L-LOC" device=""/>
-<part name="ECOG" library="eCogs" deviceset="ECOG_BUSES_ROW" device="ECOG_BUSES_SMD" value="ECOG_BUSES_ROWECOG_BUSES_SMD"/>
+<part name="ECOG" library="eCogs" deviceset="ECOG_BUSES_ROW" device="THROUGHHOLE" value="ECOG_BUSES_ROWTHROUGHHOLE"/>
 <part name="GND1" library="eCogs" deviceset="GND" device=""/>
 <part name="3V3_PWR1" library="eCogs" deviceset="3V3" device=""/>
