File: hardware/eCogs/pCog104_Tester.sch (EAGLE design)
At the start: 17 parts

Commit message: Update eCogs to through hole
Parts:
- removed S1, S2, S3, S4: (no value), SparkFun:TAC_SWITCHPTH
- added ECOG1, ECOG2, ECOG3, ECOG5: ECOG_BUSES_ROWTHROUGHHOLE, eCogs:ECOG_BUSES_ROWTHROUGHHOLE
- added ECOG4: ECOG_GENERAL_ROWTHROUGHOLE, eCogs:ECOG_GENERAL_ROWTHROUGHOLE
- added GB0, GB1, GB10, GB11, GB2, GB3, GB4, GB5, GB6, GB7, GB8, GB9, SPI-CSA, SPI-CSB, SPI-CSC, SPI-CSD, SPI-MISO, SPI-MOSI, SPI-SCK: (no value), adafruit:LEDCHIP-LED0805
- added ISP1: AVRISP-6, adafruit:AVRISP-6
- added JP1: .96 I2C OLED LCD, pinhead:PINHD-1X4
- added R10, R11, R12, R13, R14, R15, R16, R17, R18, R19, R20, R21, R22, R23, R9: 390, GadgetFactory:R0805
- ECOG: PARTNO (none) -> NREC010SABC-M30RC,SULLINS CONNECTOR SOLUTIONS,dk,S1013EC-10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
- GB12, GB13, GB14, GB15: PARTNO (none) -> LTST-C170KGKT,LITE-ON INC (VA),DK,160-1414-1-ND,LED GREEN C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
- R1, R3, R5, R7: PARTNO (none) -> MCR10EZPJ391,ROHM SEMICONDUCTOR (PASSIVE) (VA),DK,RHM390ARC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
- R2, R4, R6, R8: value 10K -> 390; DIGIKEY RMCF0805JT10K0CT-ND -> RMCF0805JT390RCT-ND; PARTNO (none) -> MCR10EZPJ391,ROHM SEMICONDUCTOR (PASSIVE) (VA),DK,RHM390ARC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
- renumbered LED1 to GB15, LED2 to GB14, LED3 to GB13, LED4 to GB12
Connections:
- removed net 1: ECOG.G0, R1A.1, R2A.2, S1.1, S1.2
- removed net 2: ECOG.G1, R3A.1, R4A.2, S2.1, S2.2
- removed net 3: ECOG.G2, R5A.1, R6A.2, S3.1, S3.2
- removed net 4: ECOG.G3, R7A.1, R8A.2, S4.1, S4.2
- new net GB0: ECOG4.G7, R20A.1
- new net GB1: ECOG4.G6, R19A.1
- new net GB10: ECOG.G5, R4A.1
- new net GB11: ECOG.G4, R2A.1
- new net GB12: ECOG.G3, R7A.1
- new net GB13: ECOG.G2, R5A.1
- new net GB14: ECOG.G1, R3A.1
- new net GB15: ECOG.G0, R1A.1
- new net GB2: ECOG4.G5, R18A.1
- new net GB3: ECOG4.G4, R17A.1
- new net GB4: ECOG4.G3, R16A.1
- new net GB5: ECOG4.G2, R15A.1
- new net GB6: ECOG4.G1, R14A.1
- new net GB7: ECOG4.G0, R13A.1
- new net GB8: ECOG.G7, R8A.1
- new net GB9: ECOG.G6, R6A.1
- new net N$10: R12A.2, SPI-MISO.A
- new net N$11: R21A.2, SPI-CSC.A
- new net N$12: GB11.A, R2A.2
- new net N$13: GB10.A, R4A.2
- new net N$14: GB9.A, R6A.2
- new net N$15: GB8.A, R8A.2
- new net N$16: GB7.A, R13A.2
- new net N$17: GB6.A, R14A.2
- new net N$18: GB5.A, R15A.2
- new net N$19: GB4.A, R16A.2
- new net N$20: GB3.A, R17A.2
- new net N$21: GB2.A, R18A.2
- new net N$22: GB1.A, R19A.2
- new net N$23: GB0.A, R20A.2
- new net N$24: R22A.2, SPI-CSD.A
- new net N$25: R23A.2, SPI-CSB.A
- new net N$26: ECOG1.SPI-CS@B3, R21A.1
- new net N$27: ECOG3.SPI-CS@B3, R22A.1
- new net N$28: ECOG5.SPI-CS@B3, R23A.1
- new net N$29: ECOG5.SPI-MISO@B0, ISP1.MISO
- new net N$30: ECOG5.SPI-SCK@B2, ISP1.SCK
- new net N$31: ECOG5.RSV@B6, ISP1.RST
- new net N$32: ECOG5.SPI-MOSI@B1, ISP1.MOSI
- new net N$5: R9A.2, SPI-CSA.A
- new net N$6: R10A.2, SPI-SCK.A
- new net N$7: ECOG2.I2C-SDA@B4, JP1.4
- new net N$8: ECOG2.I2C-SCL@B5, JP1.3
- new net N$9: R11A.2, SPI-MOSI.A
- new net SPI-CSA: ECOG2.SPI-CS@B3, R9A.1
- new net SPI-MISO: ECOG2.SPI-MISO@B0, R12A.1
- new net SPI-MOSI: ECOG2.SPI-MOSI@B1, R11A.1
- new net SPI-SCK: ECOG2.SPI-SCK@B2, R10A.1
- net 3V3: now also ECOG2.3V3@B8, ECOG4.3V3, ISP1.VCC, JP1.1; no longer S1.3, S1.4, S2.3, S2.4, S3.3, S3.4, S4.3, S4.4
- net GND: now also ECOG2.GND@B, ECOG4.GND, GB0.C, GB1.C, GB10.C, GB11.C, GB2.C, GB3.C, GB4.C, GB5.C, GB6.C, GB7.C, GB8.C, GB9.C, ISP1.GND, JP1.2, SPI-CSA.C, SPI-CSB.C, SPI-CSC.C, SPI-CSD.C, SPI-MISO.C, SPI-MOSI.C, SPI-SCK.C; no longer R2A.1, R4A.1, R6A.1, R8A.1
Other:
- note added: "Copyright 2012 Gadget Factory, LLC"
- note added: "TODO: SPI PROGRAMMER"
- note added: "This work is licensed under the Creative Commons Non-Commercial Attribution License."
