File: eCog_Templates/eCog_General_Template.sch (EAGLE design)
At the start: 1 part

Commit message: Change to through hole and give bette descriptions.
Parts:
- ECOG: value ECOG_GENERAL_ROWECOG_GENERAL_SMD -> ECOG_GENERAL_ROWTHROUGHOLE; device eCogs:ECOG_GENERAL_ROWECOG_GENERAL_SMD -> eCogs:ECOG_GENERAL_ROWTHROUGHOLE
Changed lines of the file:
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@@
 <parts>
 <part name="FRAME1" library="frames" deviceset="A3L-LOC" device=""/>
-<part name="ECOG" library="eCogs" deviceset="ECOG_GENERAL_ROW" device="ECOG_GENERAL_SMD" value="ECOG_GENERAL_ROWECOG_GENERAL_SMD"/>
+<part name="ECOG" library="eCogs" deviceset="ECOG_GENERAL_ROW" device="THROUGHOLE" value="ECOG_GENERAL_ROWTHROUGHOLE"/>
 <part name="3V3_PWR1" library="eCogs" deviceset="3V3" device=""/>
 <part name="GND1" library="eCogs" deviceset="GND" device=""/>
