File: hardware/GadgetBox-ESP8266/Gadget-Box-ESP8266-Modules.sch (EAGLE design)
At the start: 21 parts

Commit message: Added battery cutouts and re-routed everything.
Parts:
- removed R10: 10K, GadgetFactory:R0805
- AH, AL, BH, BL: value ECOGECOG_SLOT_ALT1 -> ECOGECOG_SLOT; device eCogs:ECOGECOG_SLOT_ALT1 -> eCogs:ECOGECOG_SLOT
Connections:
- net 3V3: no longer R10A.2
- net 5V0: now also AH.5V@B7, AL.5V@B7, BH.5V@B7, BL.5V@B7; no longer AH.5V@0, AL.5V@0, BH.5V@0, BL.5V@0
- net RESET: now also AH.RESET@B6, AL.RESET@B6, BH.RESET@B6, BL.RESET@B6; no longer AH.RESET@1, AL.RESET@1, BH.RESET@1, BL.RESET@1, R10A.1
Other:
- note added: "AutoReset"
