File: hardware/GadgetBox-328pb/Gadget-Box-328pb-V1.0-eagle/Gadget-Box-328pb.brd (EAGLE design)
At the start: 93.5 x 53.5 mm, 33 parts, among them U1 MCP73831T-2ACI/OT, U2 AP2112-3.3

Commit message: Misc changes for manufacturing.
Parts:
- removed D2: MBR120, microbuilder:SOD-123
- removed R11, R12, R8, R9: 10K, GadgetFactory:0805
- removed R13: 0, GadgetFactory:0805
- removed X2: (no value), adafruit:ESP-12
- added C12, C8: .1uF, we-rcl:C0805
- added C9: 100n, we-rcl:C0805
- added IC1A: ATMEGA328PB-AU, we-chip:TQFP32
- added IC1B: ATMEGA328PB-MU, we-chip:QFN32-PAD
- added L1: 10u, we-rcl:C0603
- added R7: 10K, GadgetFactory:0603
- added X1: CRYSTAL-0500290P1, OPL Eagle Library:2P-SMD-5.0X3.2
- AH, AL, BH, BL: value ECOGECOG_SLOT -> ECOGECOG_SLOT_ALT1; device eCogs:ECOG -> eCogs:ECOG_ALT1
- C11: device GadgetFactory:0805 -> we-rcl:C0603
- R10: value 10K -> 10k; device GadgetFactory:0805 -> we-rcl:C0603
- R4, R6: device GadgetFactory:0805 -> GadgetFactory:0603
- moved R4 33.6 mm to (70.1, 26.2), turned to 0 degrees
- moved JP1 2.33 mm to (15.6, 52.1), turned to 180 degrees
- moved R10 1.14 mm to (53.8, 41.1), turned to 90 degrees
- moved C11 0.38 mm to (53.8, 42.4), turned to 90 degrees
Connections:
- removed net ADC: R3.1, X2.2
- removed net D2: AL.G2, BH.G5, BH.SPI-CS@B3, X2.14
- removed net D3: AL.G3, AL.SPI-CS@B3, BH.G4, X2.13
- removed net I2C-SDA/BOOTLOAD: AH.I2C-SDA@B4, AL.I2C-SDA@B4, BH.I2C-SDA@B4, BL.I2C-SDA@B4, D2.A, R4.1, X2.12
- removed net RESET_NOTUSED: R11.1, X2.1
- removed net SPI-CSD: AH.SPI-CS@B3, X2.4
- removed net VCC: R4.2
- new net AREF: C9.2, IC1A.20, IC1B.20
- new net AVCC: C8.2, IC1A.18, IC1B.18, L1.1
- new net D10/A5: AH.G2, BL.G5, IC1A.22, IC1B.22
- new net D11*: AH.G3, BL.G4, IC1A.13, IC1B.13
- new net D12*: AH.G4, BL.G3, IC1A.9, IC1B.9
- new net D13*: AH.G5, BL.G2, IC1A.14, IC1B.14
- new net D14: AH.G6, BL.G1, IC1A.12, IC1B.12
- new net D15: AH.G7, BL.G0, IC1A.11, IC1B.11
- new net D2*: AL.G2, BH.G5, IC1A.32, IC1B.32
- new net D3*: AL.G3, BH.G4, IC1A.1, IC1B.1
- new net D4*: AL.G4, BH.G3, IC1A.10, IC1B.10
- new net D5/A0: AL.G5, BH.G2, IC1A.26, IC1B.26, R3.1
- new net D6/A1: AL.G6, BH.G1, IC1A.25, IC1B.25
- new net D7/A2: AL.G7, BH.G0, IC1A.24, IC1B.24
- new net D8/A3: AH.G0, AH.SPI-CS@B3, BL.G7, IC1A.23, IC1B.23
- new net D9/A4: AH.G1, BL.G6, IC1A.19, IC1B.19
- new net I2C-SDA: AH.I2C-SDA@B4, AL.I2C-SDA@B4, BH.I2C-SDA@B4, BL.I2C-SDA@B4, IC1A.27, IC1B.27, R4.1
- new net SPI-CSA: BH.SPI-CS@B3, IC1A.3, IC1B.3
- new net SPI-CSB: AL.SPI-CS@B3, IC1A.2, IC1B.2
- net 3V3: now also C12.2, FTDI.4, IC1A.4, IC1B.4, L1.2, R4.2, R7.2; no longer R11.2, R12.2, R13.2, R8.2, X2.8
- net 5V0: now also AH.5V@2, AL.5V@2, BH.5V@2, BL.5V@2; no longer AH.5V@B7, AL.5V@B7, BH.5V@B7, BL.5V@B7
- net D0/RX/MISO: now also IC1A.30, IC1B.30; no longer X2.15
- net D1/TX/MOSI: now also IC1A.31, IC1B.31; no longer X2.16
- net DTR: no longer D2.C
- net GND: now also C12.1, C8.1, C9.1, IC1A.21, IC1A.5, IC1B.21, IC1B.5; no longer R9.1, X2.9
- net I2C-SCL: now also IC1A.28, IC1B.28, R7.1; no longer R8.1, X2.11
- net N$5: now also IC1A.8, IC1B.8, X1.1; no longer AL.G7
- net N$6: now also IC1A.7, IC1B.7, X1.2; no longer FTDI.4, R13.1
- net RESET: now also AH.RESET@2, AL.RESET@2, BH.RESET@2, BL.RESET@2, IC1A.29, IC1B.29; no longer AH.RESET@B6, AL.RESET@B6, BH.RESET@B6, BL.RESET@B6, R12.1, X2.3
- net SPI-CSC: now also IC1A.6, IC1B.6; no longer R9.2, X2.10
- net SPI-MISO: now also IC1A.16, IC1B.16; no longer X2.6
- net SPI-MOSI: now also IC1A.15, IC1B.15; no longer X2.7
- net SPI-SCK: now also IC1A.17, IC1B.17; no longer X2.5
Routing:
- net I2C-SDA/BOOTLOAD: track 239.2 -> 0.00 mm, vias 5 -> 0
- net I2C-SDA: track 0.00 -> 179.8 mm, vias 0 -> 5
- net D2: track 109.6 -> 0.00 mm, vias 1 -> 0
- net D8/A3: track 0.00 -> 105.4 mm, vias 0 -> 3
- net D4*: track 0.00 -> 99.2 mm, vias 0 -> 3
- net D3: track 98.8 -> 0.00 mm, vias 1 -> 0
- net D15: track 0.00 -> 98.8 mm, vias 0 -> 1
- net D5/A0: track 0.00 -> 94.8 mm, vias 0 -> 1
- net D14: track 0.00 -> 94.6 mm, vias 0 -> 1
- net D12*: track 0.00 -> 92.5 mm, vias 0 -> 1
- net D2*: track 0.00 -> 92.3 mm, vias 0 -> 1
- net D13*: track 0.00 -> 90.2 mm, vias 0 -> 1
- net D3*: track 0.00 -> 87.8 mm, vias 0 -> 1
- net D10/A5: track 0.00 -> 86.3 mm, vias 0 -> 1
- net D11*: track 0.00 -> 86.0 mm, vias 0 -> 1
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Other:
- board text added: "Gadget Box - ATmega328PB Copyright 2016 Gadget Factory, LLC Version 1.0"
- board text removed: "<-Cutout"
- board text removed: "Gadget Box - ESP8266 Copyright 2016 Gadget Factory, LLC Version 1.2"
